File: FMC_Carrier_Conn.sch (KiCad schematic (older format))
At the start: 1 part, among them J1 ASP-134486-01

Commit message: Update May --> See Update Note
Parts:
- added C46, C47, C48, C49: 0.1uF, Capacitor_SMD:C_0402_1005Metric, symbol Device:C
- added IC17: 74AVC4T245RSVR-NT, ApotheoTech_CXP_Lib:74AVC4T245RSVR-NT, symbol ApotheoTech:74AVC4T245RSVR-NT
- added IC21: MC74VHC1GT66, ApotheoTech_CXP_Lib:SN74CB3T1G125DBVR, symbol ApotheoTech:MC74VHC1GT66
- added R36: 4.7K, Resistor_SMD:R_0402_1005Metric, symbol Device:R
- added U6: SN74AXC1T45DCKR, ApotheoTech_CXP_Lib:SN74AXC1T45DCKR, symbol ApotheoTech:SN74AXC1T45DCKR
Connections:
- net FMC_3V3: now also IC21.5 (VCC)
- net FMC_TCK: now also IC17.13 (2B1)
- net FMC_TDI: now also IC17.14 (1B2), IC21.1 (A)
- net FMC_TDO: now also IC21.2 (B), U6.3 (A)
- net FMC_TMS: now also IC17.15 (1B1)
- net GND: now also C46.1, C47.2, C48.2, C49.2, IC17.1 (1~OE), IC17.10 (GND_1), IC17.11 (GND_2), IC17.16 (2~OE), IC21.3 (GND), R36.1, U6.2 (GND)
- net PRSNT_M2C_B: now also IC21.4 (OE)
- new net: R36.2, U6.5 (DIR)
- new net FMC_TCK_1V8: IC17.8 (2A1)
- new net FMC_TDI_1V8: IC17.7 (1A2)
- new net FMC_TDO_FMC_1V8: U6.4 (B)
- new net FMC_TMS_1V8: IC17.6 (1A1)
- new net PS_1V8: C46.2, C48.1, IC17.3 (V_CCA), IC17.4 (1DIR), IC17.5 (2DIR), IC17.9 (2A2), U6.6 (VCCB)
- new net UTIL_3V3: C47.1, C49.1, IC17.2 (V_CCB), U6.1 (VCCA)
- no-connect marks 131 -> 132
Other:
- note added: "Bus switch to automatically short FMC TDI to TDO\nif PRSRST is not low (FMC attached)"
- note added: "DIR is high, goes from A to B\nReferenced from VCCA"
- note added: "JTAG Voltage Level Shifter (1.8V to 3.3V)"

Commit message: Pre-Production Push
Parts:
- IC21: footprint ApotheoTech_CXP_Lib:SN74CB3T1G125DBVR -> ApotheoTech_CXP_Lib:M74VHC1GT66
Connections:
- net GND: no longer R36.1
- net UTIL_3V3: now also R36.1
- net CLK0_M2C_N renamed HPC_CLK0_CLK0_M2C_N
- net CLK0_M2C_P renamed HPC_CLK0_CLK0_M2C_P
- net CLK1_M2C_N renamed HPB_CLK0_CLK1_M2C_N
- net CLK1_M2C_P renamed HPB_CLK0_CLK1_M2C_P
- net FMC_TDI_1V8 renamed FPGA_JTAG_TDO_FMC_TDI_1V8
- net FMC_TDO_FMC_1V8 renamed FMC_JTAG_TDO_1V8
- net GBTCLK0_M2C_N renamed GTH_REFCLK1_C2M_GBTCLK0_M2C_N
- net GBTCLK0_M2C_P renamed GTH_REFCLK1_C2M_GBTCLK0_M2C_P
- net LA00_CC_N renamed HPB09_LA00_CC_N
- net LA00_CC_P renamed HPB09_LA00_CC_P
- net LA01_CC_N renamed HPB15_CC_LA01_CC_N
- net LA01_CC_P renamed HPB15_CC_LA01_CC_P
- net LA02_N renamed HPB10_CC_LA02_N
- net LA02_P renamed HPB10_CC_LA02_P
- net LA03_N renamed HPB07_LA03_N
- net LA03_P renamed HPB07_LA03_P
- net LA04_N renamed HPB08_LA04_N
- net LA04_P renamed HPB08_LA04_P
- net LA05_N renamed HPB14_LA05_N
- net LA05_P renamed HPB14_LA05_P
- net LA06_N renamed HPB01_LA06_N
- net LA06_P renamed HPB01_LA06_P
- net LA07_N renamed HPB02_LA07_N
- net LA07_P renamed HPB02_LA07_P
- net LA08_N renamed HPB00_CC_LA08_N
- net LA08_P renamed HPB00_CC_LA08_P
- net LA09_N renamed HPB12_LA09_N
- net LA09_P renamed HPB12_LA09_P
- net LA10_N renamed HPB05_CC_LA10_N
- net LA10_P renamed HPB05_CC_LA10_P
- net LA11_N renamed HPB13_LA11_N
- net LA11_P renamed HPB13_LA11_P
- net LA12_N renamed HPB04_LA12_N
- net LA12_P renamed HPB04_LA12_P
- net LA13_N renamed HPB06_LA13_N
- net LA13_P renamed HPB06_LA13_P
- net LA14_N renamed HPB11_LA14_N
- net LA14_P renamed HPB11_LA14_P
- net LA15_N renamed HPB18_LA15_N
- net LA15_P renamed HPB18_LA15_P
- net LA16_N renamed HPB16_LA16_N
- net LA16_P renamed HPB16_LA16_P
- net LA17_CC_N renamed HPB17_LA17_CC_N
- net LA17_CC_P renamed HPB17_LA17_CC_P
- net LA18_CC_N renamed HPC08_LA18_CC_N
- net LA18_CC_P renamed HPC08_LA18_CC_P
- net LA19_N renamed HPB19_LA19_N
- net LA19_P renamed HPB19_LA19_P
- net LA20_N renamed HPB03_LA20_N
- net LA20_P renamed HPB03_LA20_P
- net LA21_N renamed HPC16_LA21_N
- net LA21_P renamed HPC16_LA21_P
- net LA22_N renamed HPC19_LA22_N
- net LA22_P renamed HPC19_LA22_P
- net LA23_N renamed HPC13_LA23_N
- net LA23_P renamed HPC13_LA23_P
- net LA24_N renamed HPC05_CC_LA24_N
- net LA24_P renamed HPC05_CC_LA24_P
- net LA25_N renamed HPC15_CC_LA25_N
- net LA25_P renamed HPC15_CC_LA25_P
- net LA26_N renamed HPC14_LA26_N
- net LA26_P renamed HPC14_LA26_P
- net LA27_N renamed HPC07_LA27_N
- net LA27_P renamed HPC07_LA27_P
- net LA28_N renamed HPC04_LA28_N
- net LA28_P renamed HPC04_LA28_P
- net LA29_N renamed HPC18_LA29_N
- net LA29_P renamed HPC18_LA29_P
- net LA30_N renamed HDB19_LA30_N
- net LA30_P renamed HDB18_LA30_P
- net LA31_N renamed HPC03_LA31_N
- net LA31_P renamed HPC03_LA31_P
- net LA32_N renamed HDB16_CC_LA32_N
- net LA32_P renamed HDB15_LA32_P
- net LA33_N renamed HDB22_LA33_N
- net LA33_P renamed HDB21_LA33_P
- net PRSNT_M2C_B renamed HDC18_PRSNT_M2C_B
- net RX_DP0_M2C_N renamed GTH_DP2_C2M_RX_DP0_M2C_N
- net RX_DP0_M2C_P renamed GTH_DP2_C2M_RX_DP0_M2C_P
- net RX_DP1_M2C_N renamed GTH_DP0_C2M_RX_DP1_M2C_N
- net RX_DP1_M2C_P renamed GTH_DP0_C2M_RX_DP1_M2C_P
- net TX_DP0_C2M_N renamed GTH_DP2_M2C_TX_DP0_C2M_N
- net TX_DP0_C2M_P renamed GTH_DP2_M2C_TX_DP0_C2M_P
- net TX_DP1_C2M_N renamed GTH_DP0_M2C_TX_DP1_C2M_N
- net TX_DP1_C2M_P renamed GTH_DP0_M2C_TX_DP1_C2M_P
- net TX_DP2_C2M_N renamed GTH_DP3_M2C_TX_DP2_C2M_N
- net TX_DP2_C2M_P renamed GTH_DP3_M2C_TX_DP2_C2M_P
- net TX_DP3_C2M_N renamed GTH_DP1_M2C_TX_DP3_C2M_N
- net TX_DP3_C2M_P renamed GTH_DP1_M2C_TX_DP3_C2M_P
Other:
- note added: "Bus switch to automatically short FMC TDI to TDO\nif PRSNT_M2C_B is not low (FMC attached)"
- note added: "DIR is high, goes from A to B\nReferenced from VCCA (3.3V here)"
- note added: "Look on right hand side:\nC2M for VITA 57.1 is TX"
- note added: "Note, switch only operates 3.3V to 5V\nThis is why we need to have switch on 3.3V side"
- note added: "Refer to page / of ZCU106 for pinout of FMC.\nOr Refer to page / of VITA 57.1 documentation"
- note removed: "Bus switch to automatically short FMC TDI to TDO\nif PRSRST is not low (FMC attached)"
