File: MIPI_Conn.sch (KiCad schematic (older format))
At the start: 8 parts, among them J13 FH12-22S-0.5SH_55_, J14 FH12-22S-0.5SH_55_

Commit message: Update May --> See Update Note
Other:
- note added: "Mipi PCB guidelines on Page 203/347 of UG 583"
Changed lines of the file:
@@
 Text GLabel 6200 4100 0    50   BiDi ~ 0
 CAM1_SDA
+Text Notes 4930 1555 0    118  ~ 0
+Mipi PCB guidelines on Page 203/347 of UG 583
 $EndSCHEMATC

Commit message: Pre-Production Push
Connections:
- net CAM0_GPIO_1 renamed HDA01_CAM0_GPIO_1
- net CAM1_GPIO_1 renamed HDC13_CAM1_GPIO_1
- net HPB05_CC_MIPI_B1_CLK_N renamed HPA05_CC_MIPI_A1_CLK_N
- net HPB05_CC_MIPI_B1_CLK_P renamed HPA05_CC_MIPI_A1_CLK_P
- net HPB06_MIPI_B1_D0_N renamed HPA06_MIPI_A1_D0_N
- net HPB06_MIPI_B1_D0_P renamed HPA06_MIPI_A1_D0_P
- net HPB07_MIPI_B1_D1_N renamed HPA07_MIPI_A1_D1_N
- net HPB07_MIPI_B1_D1_P renamed HPA07_MIPI_A1_D1_P
- net HPB08_MIPI_B1_D2_N renamed HPA08_MIPI_A1_D2_N
- net HPB08_MIPI_B1_D2_P renamed HPA08_MIPI_A1_D2_P
- net HPB09_MIPI_B1_D3_N renamed HPA09_MIPI_A1_D3_N
- net HPB09_MIPI_B1_D3_P renamed HPA09_MIPI_A1_D3_P
Other:
- note added: "Referenced from https://www.arducam.com/raspberry-pi-camera-pinout/\nAnd from CM4IOV5 schematic for MIPI connectors"
Changed lines of the file:
@@
 $Descr A4 11693 8268
 encoding utf-8
-Sheet 8 20
+Sheet 20 20
 Title "MIPI DSI and CSI-2 Connectors"
 Date "2022-01-04"
@@
 Text HLabel 2200 3400 0    50   Output ~ 0
 HPA04_MIPI_A0_D3_N
-Text HLabel 2200 3800 0    50   Input ~ 0
-CAM0_GPIO_1
+Text HLabel 2200 3800 0    39   Input ~ 0
+HDA01_CAM0_GPIO_1
 Wire Wire Line
 	2250 3800 2200 3800
@@
 Text HLabel 5400 3700 0    50   Input ~ 0
 CAM1_RESET_N
-Text HLabel 6200 3800 0    50   Input ~ 0
-CAM1_GPIO_1
+Text HLabel 6200 3800 0    39   Input ~ 0
+HDC13_CAM1_GPIO_1
 Wire Wire Line
 	6250 3800 6200 3800
@@
 $EndComp
 Text HLabel 6200 3500 0    50   Output ~ 0
-HPB09_MIPI_B1_D3_P
+HPA09_MIPI_A1_D3_P
 Text HLabel 6200 3400 0    50   Output ~ 0
-HPB09_MIPI_B1_D3_N
+HPA09_MIPI_A1_D3_N
 Text HLabel 6200 3200 0    50   Output ~ 0
-HPB08_MIPI_B1_D2_P
+HPA08_MIPI_A1_D2_P
 Text HLabel 6200 3100 0    50   Output ~ 0
-HPB08_MIPI_B1_D2_N
+HPA08_MIPI_A1_D2_N
 Text HLabel 6200 2300 0    50   Output ~ 0
-HPB06_MIPI_B1_D0_P
+HPA06_MIPI_A1_D0_P
 Text HLabel 6200 2200 0    50   Output ~ 0
-HPB06_MIPI_B1_D0_N
+HPA06_MIPI_A1_D0_N
 Text HLabel 6200 2800 0    50   Output ~ 0
-HPB05_CC_MIPI_B1_CLK_N
+HPA05_CC_MIPI_A1_CLK_N
 Text HLabel 6200 2900 0    50   Output ~ 0
-HPB05_CC_MIPI_B1_CLK_P
+HPA05_CC_MIPI_A1_CLK_P
 Text Label 6200 4100 0    50   ~ 0
 CAM1_SDA
@@
 	6700 2800 6200 2800
 Text HLabel 6200 2600 0    50   Output ~ 0
-HPB07_MIPI_B1_D1_P
+HPA07_MIPI_A1_D1_P
 Text HLabel 6200 2500 0    50   Output ~ 0
-HPB07_MIPI_B1_D1_N
+HPA07_MIPI_A1_D1_N
 Wire Wire Line
 	6700 2600 6200 2600
@@
 Text Notes 4930 1555 0    118  ~ 0
 Mipi PCB guidelines on Page 203/347 of UG 583
+Text Notes 4885 945  0    50   ~ 0
+Referenced from https://www.arducam.com/raspberry-pi-camera-pinout/\nAnd from CM4IOV5 schematic for MIPI connectors
 $EndSCHEMATC
