File: SOM240_1.sch (KiCad schematic (older format))
At the start: 2 parts, among them J17 ADM6-60-01.5-L-4-2-A-TR

Commit message: Pre-Production Push
Connections:
- net HDA01 renamed HDA01_CAM0_GPIO_1
- net HDA02 renamed HDA02_DP_PWR_EN
- net HDA12 renamed HDA12_DP_PWR_FAULT
- net HDA19 renamed HDA19_ALERT_INA260
- net HDA20_FAN renamed HDA20
- net HPA10_CC_MIPI_A2_CLK_N renamed HPA10_CC_N
- net HPA10_CC_MIPI_A2_CLK_P renamed HPA10_CC_P
- net HPA11_MIPI_A2_D0_N renamed HPA11_N
- net HPA11_MIPI_A2_D0_P renamed HPA11_P
- net HPA12_MIPI_A2_D1_N renamed HPA12_N
- net HPA12_MIPI_A2_D1_P renamed HPA12_P
- net HPA13_MIPI_A2_D2_N renamed HPA13_N
- net HPA13_MIPI_A2_D2_P renamed HPA13_P
- net HPA14_MIPI_A2_D3_N renamed HPA14_N
- net HPA14_MIPI_A2_D3_P renamed HPA14_P
- net JTAG_TCK_C2M renamed FPGA_JTAG_TCK_C2M_1V8
- net JTAG_TDI_C2M renamed FPGA_JTAG_TDI_C2M_1V8
- net JTAG_TDO_M2C renamed FPGA_JTAG_TDO_FMC_TDI_1V8
- net JTAG_TMS_C2M renamed FPGA_JTAG_TMS_C2M_1V8
- net MIO64_SPI0_SCLK renamed MIO64
- net MIO67_SPI0_CS_N renamed MIO67
- net MIO68_SPI0_MISO renamed MIO68
- net MIO69_SPI0_MOSI renamed MIO69
- net MIO70_UART_RXD renamed MIO70
- net MIO71_UART_TXD renamed MIO71
Other:
- note added: "VCCO_HDA (3.3V)"
- note added: "VCC_HPA (1.2V for MIPI)"
Changed lines of the file:
@@
 $Descr A3 16535 11693
 encoding utf-8
-Sheet 11 20
+Sheet 10 20
 Title "SOM240-1"
 Date "2022-01-04"
@@
 	2450 3350 2900 3350
 Text HLabel 2900 3350 2    50   Input ~ 0
-HPA12_MIPI_A2_D1_P
+HPA12_P
 Wire Wire Line
 	2450 3450 2900 3450
 Text HLabel 2900 3450 2    50   Input ~ 0
-HPA12_MIPI_A2_D1_N
+HPA12_N
 Wire Wire Line
 	2450 3950 2900 3950
@@
 	2450 4650 2900 4650
 Text HLabel 2900 4650 2    50   Input ~ 0
-JTAG_TMS_C2M
+FPGA_JTAG_TMS_C2M_1V8
 Wire Wire Line
 	2450 4750 2900 4750
 Text HLabel 2900 4750 2    50   Output ~ 0
-JTAG_TDO_M2C
+FPGA_JTAG_TDO_FMC_TDI_1V8
 Wire Wire Line
 	2450 4850 2900 4850
 Text HLabel 2900 4850 2    50   Input ~ 0
-JTAG_TDI_C2M
+FPGA_JTAG_TDI_C2M_1V8
 Wire Wire Line
 	2450 4950 2900 4950
 Text HLabel 2900 4950 2    50   Input ~ 0
-JTAG_TCK_C2M
+FPGA_JTAG_TCK_C2M_1V8
 Wire Wire Line
 	2450 5150 2900 5150
@@
 HPA07_MIPI_A1_D1_N
 Text HLabel 5900 3450 2    50   Input ~ 0
-HPA11_MIPI_A2_D0_P
+HPA11_P
 Text HLabel 5900 3550 2    50   Input ~ 0
-HPA11_MIPI_A2_D0_N
+HPA11_N
 Text HLabel 5900 4050 2    50   Input ~ 0
 HDA03
@@
 MIO58_USB_STP
 Text HLabel 5900 6850 2    50   Input ~ 0
-MIO70_UART_RXD
+MIO70
 Text HLabel 5900 6950 2    50   Output ~ 0
-MIO71_UART_TXD
+MIO71
 Text HLabel 5900 7050 2    50   Input ~ 0
 MIO72
@@
 HPA02_MIPI_A0_D1_N
 Text HLabel 11900 3750 2    50   Input ~ 0
-HPA14_MIPI_A2_D3_P
+HPA14_P
 Text HLabel 11900 3850 2    50   Input ~ 0
-HPA14_MIPI_A2_D3_N
+HPA14_N
 Text HLabel 11900 4050 2    50   Input ~ 0
 HDA00_CC
-Text HLabel 11900 4150 2    50   Input ~ 0
-HDA01
-Text HLabel 11900 4250 2    50   Input ~ 0
-HDA02
+Text HLabel 11900 4150 2    50   Output ~ 0
+HDA01_CAM0_GPIO_1
+Text HLabel 11900 4250 2    50   Output ~ 0
+HDA02_DP_PWR_EN
 Text HLabel 11900 4550 2    50   Input ~ 0
 HDA13
@@
 MIO54_USB_DATA2
 Text HLabel 11900 6450 2    50   Output ~ 0
-MIO64_SPI0_SCLK
+MIO64
 Text HLabel 11900 6850 2    50   Input ~ 0
 MIO76
@@
 	2450 3650 2900 3650
 Text HLabel 2900 3650 2    50   Input ~ 0
-HPA13_MIPI_A2_D2_P
+HPA13_P
 Wire Wire Line
 	2450 3750 2900 3750
 Text HLabel 2900 3750 2    50   Input ~ 0
-HPA13_MIPI_A2_D2_N
+HPA13_N
 Wire Wire Line
 	2600 3550 2600 3850
@@
 	8450 4750 8900 4750
 Text HLabel 8900 4750 2    50   Input ~ 0
-HDA19
+HDA19_ALERT_INA260
 Wire Wire Line
 	8450 5050 8900 5050
@@
 	8450 3650 8900 3650
 Text HLabel 8900 3650 2    50   Input ~ 0
-HPA10_CC_MIPI_A2_CLK_P
+HPA10_CC_P
 Wire Wire Line
 	8450 3750 8900 3750
 Text HLabel 8900 3750 2    50   Input ~ 0
-HPA10_CC_MIPI_A2_CLK_N
+HPA10_CC_N
 Wire Wire Line
 	8600 3550 8600 3850
@@
 	8450 6650 8900 6650
 Text HLabel 8900 6650 2    50   Output ~ 0
-MIO67_SPI0_CS_N
+MIO67
 Wire Wire Line
 	8450 6750 8900 6750
 Text HLabel 8900 6750 2    50   Input ~ 0
-MIO68_SPI0_MISO
+MIO68
 Wire Wire Line
 	8450 6850 8900 6850
 Text HLabel 8900 6850 2    50   Output ~ 0
-MIO69_SPI0_MOSI
+MIO69
 Wire Wire Line
 	8450 7850 8600 7850
@@
 	8450 4850 8900 4850
 Text HLabel 8900 4850 2    50   Output ~ 0
-HDA20_FAN
+HDA20
 Wire Wire Line
 	8600 3850 8600 4150
@@
 	11600 4350 11600 4750
 Text HLabel 11900 4450 2    50   Input ~ 0
-HDA12
+HDA12_DP_PWR_FAULT
 Wire Wire Line
 	11450 4450 11900 4450
@@
 Text GLabel 5900 3850 2    50   Input ~ 0
 PL_3V3
+Text Notes 6320 3855 0    50   ~ 0
+VCCO_HDA (3.3V)
+Text Notes 12395 2635 0    50   ~ 0
+VCC_HPA (1.2V for MIPI)
 $EndSCHEMATC
