File: SOM240_2.sch (KiCad schematic (older format))
At the start: 1 part, among them J3 ADM6-60-01.5-L-4-2-A-TR

Commit message: Pre-Production Push
Connections:
- net GTH_DP0_C2M_SLVS_EC_RX_N renamed GTH_DP0_C2M_RX_DP1_M2C_N
- net GTH_DP0_C2M_SLVS_EC_RX_P renamed GTH_DP0_C2M_RX_DP1_M2C_P
- net GTH_DP0_M2C_N renamed GTH_DP0_M2C_TX_DP1_C2M_N
- net GTH_DP0_M2C_P renamed GTH_DP0_M2C_TX_DP1_C2M_P
- net GTH_DP1_C2M_SLVS_EC_RX_N renamed GTH_DP1_C2M_SLVS_EC_RX_LANE1_N
- net GTH_DP1_C2M_SLVS_EC_RX_P renamed GTH_DP1_C2M_SLVS_EC_RX_LANE1_P
- net GTH_DP1_M2C_N renamed GTH_DP1_M2C_TX_DP3_C2M_N
- net GTH_DP1_M2C_P renamed GTH_DP1_M2C_TX_DP3_C2M_P
- net GTH_DP2_C2M_CXP_HOST_RX_N renamed GTH_DP2_M2C_TX_DP0_C2M_N
- net GTH_DP2_C2M_CXP_HOST_RX_P renamed GTH_DP2_M2C_TX_DP0_C2M_P
- net GTH_DP2_M2C_CXP_DEV_TX_N renamed GTH_DP2_C2M_RX_DP0_M2C_N
- net GTH_DP2_M2C_CXP_DEV_TX_P renamed GTH_DP2_C2M_RX_DP0_M2C_P
- net GTH_DP3_C2M_SDI_RX_N renamed GTH_DP3_C2M_SLVS_EC_RX_LANE0_N
- net GTH_DP3_C2M_SDI_RX_P renamed GTH_DP3_C2M_SLVS_EC_RX_LANE0_P
- net GTH_DP3_M2C_SDI_TX_N renamed GTH_DP3_M2C_TX_DP2_C2M_N
- net GTH_DP3_M2C_SDI_TX_P renamed GTH_DP3_M2C_TX_DP2_C2M_P
- net GTH_REFCLK1_C2M_N renamed GTH_REFCLK1_C2M_GBTCLK0_M2C_N
- net GTH_REFCLK1_C2M_P renamed GTH_REFCLK1_C2M_GBTCLK0_M2C_P
- net HDB03_CAM0_RESET_N renamed HDB03
- net HDB04_CAM0_RESET_N renamed HDB04
- net HDB15 renamed HDB15_LA32_P
- net HDB16_CC renamed HDB16_CC_LA32_N
- net HDB18 renamed HDB18_LA30_P
- net HDB19 renamed HDB19_LA30_N
- net HDB21 renamed HDB21_LA33_P
- net HDB22 renamed HDB22_LA33_N
- net HDC00_CC renamed HDC00_CC_INT_ICM_42688
- net HDC01 renamed HDC01_SDO_ICM_42688
- net HDC02 renamed HDC02_SDI_ICM_42688
- net HDC03 renamed HDC03_CLK_ICM_42688
- net HDC04_24V_BOOST_EN_CXP renamed HDC04_SDA_SDI_MS5611
- net HDC05_24V_DC_EN_R renamed HDC05_SCL_MS5611
- net HDC06 renamed HDC06_CAM1_RESET_N
- net HDC07 renamed HDC07_SCLK_ICM_42688
- net HDC08_CC renamed HDC08_CS_ICM_42688
- net HDC09_ALERT_PAC1720 renamed HDC09_FAN_PWM
- net HDC10_SDA_PAC1720 renamed HDC10_SDO_MS5611
- net HDC11_SCL_PAC1720 renamed HDC11_CS_MS5611
- net HDC13 renamed HDC13_CAM1_GPIO_1
- net HDC14 renamed HDC14_CAM0_RESET_N
- net HDC18 renamed HDC18_PRSNT_M2C_B
- net HDC19 renamed HDC19_INA226_ALERT
- net HDC20 renamed HDC20_VADJ_ALERT
- net HDC23 renamed HDC23_MODE_MS5611
- net HPB00_CC_MIPI_B0_CLK_N renamed HPB00_CC_LA08_N
- net HPB00_CC_MIPI_B0_CLK_P renamed HPB00_CC_LA08_P
- net HPB01_MIPI_B0_D0_N renamed HPB01_LA06_N
- net HPB01_MIPI_B0_D0_P renamed HPB01_LA06_P
- net HPB02_MIPI_B0_D1_N renamed HPB02_LA07_N
- net HPB02_MIPI_B0_D1_P renamed HPB02_LA07_P
- net HPB03_MIPI_B0_D2_N renamed HPB03_LA20_N
- net HPB03_MIPI_B0_D2_P renamed HPB03_LA20_P
- net HPB04_MIPI_B0_D3_N renamed HPB04_LA12_N
- net HPB04_MIPI_B0_D3_P renamed HPB04_LA12_P
- net HPB05_CC_MIPI_B1_CLK_N renamed HPB05_CC_LA10_N
- net HPB05_CC_MIPI_B1_CLK_P renamed HPB05_CC_LA10_P
- net HPB06_MIPI_B1_D0_N renamed HPB06_LA13_N
- net HPB06_MIPI_B1_D0_P renamed HPB06_LA13_P
- net HPB07_MIPI_B1_D1_N renamed HPB07_LA03_N
- net HPB07_MIPI_B1_D1_P renamed HPB07_LA03_P
- net HPB08_MIPI_B1_D2_N renamed HPB08_LA04_N
- net HPB08_MIPI_B1_D2_P renamed HPB08_LA04_P
- net HPB09_MIPI_B1_D3_N renamed HPB09_LA00_CC_N
- net HPB09_MIPI_B1_D3_P renamed HPB09_LA00_CC_P
- net HPB10_CC_N renamed HPB10_CC_LA02_N
- net HPB10_CC_P renamed HPB10_CC_LA02_P
- net HPB11_N renamed HPB11_LA14_N
- net HPB11_P renamed HPB11_LA14_P
- net HPB12_N renamed HPB12_LA09_N
- net HPB12_P renamed HPB12_LA09_P
- net HPB13_N renamed HPB13_LA11_N
- net HPB13_P renamed HPB13_LA11_P
- net HPB14_N renamed HPB14_LA05_N
- net HPB14_P renamed HPB14_LA05_P
- net HPB15_CC_N renamed HPB15_CC_LA01_CC_N
- net HPB15_CC_P renamed HPB15_CC_LA01_CC_P
- net HPB16_N renamed HPB16_LA16_N
- net HPB16_P renamed HPB16_LA16_P
- net HPB17_N renamed HPB17_LA17_CC_N
- net HPB17_P renamed HPB17_LA17_CC_P
- net HPB18_N renamed HPB18_LA15_N
- net HPB18_P renamed HPB18_LA15_P
- net HPB19_N renamed HPB19_LA19_N
- net HPB19_P renamed HPB19_LA19_P
- net HPB_CLK0_N renamed HPB_CLK0_CLK1_M2C_N
- net HPB_CLK0_P renamed HPB_CLK0_CLK1_M2C_P
- net HPC03_N renamed HPC03_LA31_N
- net HPC03_P renamed HPC03_LA31_P
- net HPC04_N renamed HPC04_LA28_N
- net HPC04_P renamed HPC04_LA28_P
- net HPC05_CC_N renamed HPC05_CC_LA24_N
- net HPC05_CC_P renamed HPC05_CC_LA24_P
- net HPC06_P_MCLK_0_SLVS renamed HPC06_P_GPIO16_SLAMODE1
- net HPC07_N renamed HPC07_LA27_N
- net HPC07_P renamed HPC07_LA27_P
- net HPC08_N renamed HPC08_LA18_CC_N
- net HPC08_P renamed HPC08_LA18_CC_P
- net HPC10_CC_P_GPIO16_SLAMODE1 renamed HPC10_CC_P_MCLK_0_SLVS
- net HPC13_N renamed HPC13_LA23_N
- net HPC13_P renamed HPC13_LA23_P
- net HPC14_N renamed HPC14_LA26_N
- net HPC14_P renamed HPC14_LA26_P
- net HPC15_CC_N renamed HPC15_CC_LA25_N
- net HPC15_CC_P renamed HPC15_CC_LA25_P
- net HPC16_N renamed HPC16_LA21_N
- net HPC16_P renamed HPC16_LA21_P
- net HPC18_N renamed HPC18_LA29_N
- net HPC18_P renamed HPC18_LA29_P
- net HPC19_N renamed HPC19_LA22_N
- net HPC19_P renamed HPC19_LA22_P
- net HPC_CLK0_N renamed HPC_CLK0_CLK0_M2C_N
- net HPC_CLK0_P renamed HPC_CLK0_CLK0_M2C_P
