File: USB-3_0.sch (KiCad schematic (older format))
At the start: 25 parts, among them IC5 USB3320C-EZK-TR, J5 GSB443133HR, U14 MIC2544-1YM-TR

Commit message: Update May --> See Update Note
Parts:
- removed D6: TPD4E05U06DQAR, ApotheoTech_CXP_Lib:TPD4E05U06DQAR, symbol ApotheoTech:TPD4E05U06DQAR
- removed D8: TPD2EUSB30DRTR, ApotheoTech_CXP_Lib:TPD2EUSB30DRTR, symbol ApotheoTech:TPD2EUSB30DRTR
- removed J5: GSB443133HR, ApotheoTech_CXP_Lib:GSB443133HR, symbol ApotheoTech:GSB443133HR
- added D2, D3, D4, D6: PESD3V3Y1BSFYL, Diode_SMD:D_0603_1608Metric, symbol Device:D_TVS
- added D8: RCLAMP0582BQTCT, ApotheoTech_CXP_Lib:RCLAMP0582BQTCT, symbol ApotheoTech:RCLAMP0582BQTCT
- added J5: 692122030100, ApotheoTech_CXP_Lib:692122030100, symbol ApotheoTech:692122030100
- C73: PartNumber (none) -> EEF-CX0J121R; URL (none) -> https://www.mouser.com/ProductDetail/Panasonic/EEF-CX0J121R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
- U14: PartNumber (none) -> MIC2544-1YM-TR
Connections:
- net ULPIO_ID is gone; now on net GND: IC5.23 (ID)
- net GND: now also D2.2 (A2), D3.2 (A2), D4.2 (A2), D6.2 (A2), D8.3 (GND), J5.7 (GND_DRAIN)
- net GT2_TX_C_N: now also D6.1 (A1), J5.8 (STDA_SSTX)
- net GT2_TX_C_P: now also D4.1 (A1), J5.9 (STDA_SSTX+)
- net GTR_DP2_C2M_USB0_RX_N: now also D3.1 (A1), J5.5 (STDA_SSRX)
- net GTR_DP2_C2M_USB0_RX_P: now also D2.1 (A1), J5.6 (STDA_SSRX+)
- net ULPI0_D_N: now also D8.2 (D-), J5.2 (D-)
- net ULPI0_D_P: now also D8.1 (D+), J5.3 (D+)
- net USB_VBUS: now also J5.1 (VBUS)
- net at C76.1, L9.1: now also J5.4 (GND)
- net at R75.1: now also J5.MH1, J5.MH2
Other:
- note added: "Package delay skews and CLK should be between +- 100PS (page 196/347) UG583"
- moved on the sheet: R75

Commit message: Pre-Production Push
Parts:
- removed C74: 0.1uF, Capacitor_SMD:C_0402_1005Metric, symbol Device:C
- removed R75: 0, Resistor_SMD:R_0402_1005Metric, symbol Device:R
- added C52: 1uF, Capacitor_SMD:C_0402_1005Metric, symbol Device:C
- added C53: 4.7uF, Capacitor_SMD:C_0402_1005Metric, symbol Device:C
- D2, D3, D4, D6: footprint Diode_SMD:D_0603_1608Metric -> Diode_SMD:D_0201_0603Metric
Connections:
- net GND: now also J5.MH1, J5.MH2, C52.1, C53.1
- net USB_VBUS_SEL: now also C52.2, C53.2
Other:
- note added: "Possibly increase resistor here for less brightness"
Changed lines of the file:
@@
-$EndComp
-$Comp
-L Device:R R?
-U 1 1 613AD852
-P 4460 4705
-AR Path="/5F71E87D/613AD852" Ref="R?"  Part="1"
-AR Path="/5F71E4A6/613AD852" Ref="R?"  Part="1"
-AR Path="/6314DEA9/613AD852" Ref="R71"  Part="1"
-F 0 "R71" V 4500 4875 50  0000 L CNN
-F 1 "160" V 4510 4450 50  0000 L CNN
-F 2 "Resistor_SMD:R_0402_1005Metric" V 4390 4705 50  0001 C CNN
-F 3 "~" H 4460 4705 50  0001 C CNN
-F 4 "1%" V 4400 4480 50  0000 L CNN "Tolerance"
-F 5 "ERJ-2RKF1600X" H 4460 4705 50  0001 C CNN "PartNumber"
-	1    4460 4705
-	0    -1   -1   0
 $EndComp
 $Comp
@@
 	6960 2850 6960 3140
 Wire Wire Line
-	7200 2850 6960 2850
+	7200 2850 7000 2850
 Connection ~ 7200 2850
 Wire Wire Line
@@
 $Comp
 L Device:C C?
-U 1 1 614E7F6B
-P 7200 3075
-AR Path="/5F71E87D/614E7F6B" Ref="C?"  Part="1"
-AR Path="/5F71E4A6/614E7F6B" Ref="C?"  Part="1"
-AR Path="/6314CDE6/614E7F6B" Ref="C?"  Part="1"
-AR Path="/6314DEA9/614E7F6B" Ref="C74"  Part="1"
-F 0 "C74" H 7040 3015 50  0000 C CNN
-F 1 "0.1uF" H 6980 3080 50  0000 C CNN
-F 2 "Capacitor_SMD:C_0402_1005Metric" H 7238 2925 50  0001 C CNN
-F 3 "~" H 7200 3075 50  0001 C CNN
-F 4 "TMK105BJ104KVHF" H 7200 3075 50  0001 C CNN "PartNumber"
-F 5 "+-10%" H 7200 3075 50  0001 C CNN "Tolerance"
-F 6 "25V" H 7015 3155 50  0000 C CNN "Voltage"
-F 7 "X5R" H 7200 3075 50  0001 C CNN "Temp_Val"
-F 8 "https://www.digikey.com/en/products/detail/TMK105BJ104KVHF/587-3808-1-ND/4811278?itemSeq=375666509" V 7200 3075 50  0001 C CNN "URL"
-	1    7200 3075
-	-1   0    0    1
-$EndComp
-$Comp
-L Device:C C?
 U 1 1 614EDFF4
 P 7750 3075
@@
 	1    0    0    -1
 $EndComp
-Wire Wire Line
-	10600 3750 10600 3800
 Text HLabel 1810 1340 0    50   Input ~ 0
 USB_RESET_N
@@
 Text HLabel 4350 1950 2    50   Input ~ 0
 USB_PHY_REFCLK
-$Comp
-L Device:R R?
-U 1 1 6171449A
-P 10600 3600
-AR Path="/5F71E4A6/6171449A" Ref="R?"  Part="1"
-AR Path="/5F71E87D/6171449A" Ref="R?"  Part="1"
-AR Path="/6314CDE6/6171449A" Ref="R?"  Part="1"
-AR Path="/6314DEA9/6171449A" Ref="R75"  Part="1"
-F 0 "R75" H 10700 3670 50  0000 C CNN
-F 1 "0" H 10675 3600 50  0000 C CNN
-F 2 "Resistor_SMD:R_0402_1005Metric" V 10530 3600 50  0001 C CNN
-F 3 "~" H 10600 3600 50  0001 C CNN
-F 4 "CRCW04020000Z0EDHP" V 10600 3600 50  0001 C CNN "PartNumber"
-F 5 "1/5W" H 10755 3535 50  0000 C CNN "Power"
-F 6 "https://www.digikey.com/product-detail/en/vishay-dale/CRCW04020000Z0EDHP/541-0-0YBCT-ND/2223008" V 10600 3600 50  0001 C CNN "URL"
-	1    10600 3600
-	1    0    0    -1
-$EndComp
 Text Notes 505  4960 0    50   ~ 0
 Package delay skews and CLK should be between +- 100PS (page 196/347) UG583
@@
 	1    0    0    -1
 $EndComp
-Wire Wire Line
-	10600 2950 10600 3450
 $Comp
 L Device:D_TVS D2
@@
 F 0 "D2" V 2928 7080 50  0000 L CNN
 F 1 "PESD3V3Y1BSFYL" V 2995 7080 20  0000 L CNN
-F 2 "Diode_SMD:D_0603_1608Metric" H 2950 7000 50  0001 C CNN
+F 2 "Diode_SMD:D_0201_0603Metric" H 2950 7000 50  0001 C CNN
 F 3 "~" H 2950 7000 50  0001 C CNN
 F 4 "PESD3V3Y1BSFYL" V 2950 7000 50  0001 C CNN "PartNumber"
@@
 F 0 "D3" V 3328 7080 50  0000 L CNN
 F 1 "PESD3V3Y1BSFYL" V 3395 7080 20  0000 L CNN
-F 2 "Diode_SMD:D_0603_1608Metric" H 3350 7000 50  0001 C CNN
+F 2 "Diode_SMD:D_0201_0603Metric" H 3350 7000 50  0001 C CNN
 F 3 "~" H 3350 7000 50  0001 C CNN
 F 4 "PESD3V3Y1BSFYL" V 3350 7000 50  0001 C CNN "PartNumber"
@@
 F 0 "D4" V 3728 7080 50  0000 L CNN
 F 1 "PESD3V3Y1BSFYL" V 3795 7080 20  0000 L CNN
-F 2 "Diode_SMD:D_0603_1608Metric" H 3750 7000 50  0001 C CNN
+F 2 "Diode_SMD:D_0201_0603Metric" H 3750 7000 50  0001 C CNN
 F 3 "~" H 3750 7000 50  0001 C CNN
 F 4 "PESD3V3Y1BSFYL" V 3750 7000 50  0001 C CNN "PartNumber"
@@
 F 0 "D6" V 4178 7080 50  0000 L CNN
 F 1 "PESD3V3Y1BSFYL" V 4245 7080 20  0000 L CNN
-F 2 "Diode_SMD:D_0603_1608Metric" H 4200 7000 50  0001 C CNN
+F 2 "Diode_SMD:D_0201_0603Metric" H 4200 7000 50  0001 C CNN
 F 3 "~" H 4200 7000 50  0001 C CNN
 F 4 "PESD3V3Y1BSFYL" V 4200 7000 50  0001 C CNN "PartNumber"
@@
 	1    0    0    -1
 $EndComp
+$Comp
+L Device:C C?
+U 1 1 62C50742
+P 7200 3075
+AR Path="/5F71E87D/62C50742" Ref="C?"  Part="1"
+AR Path="/5F71E4A6/62C50742" Ref="C?"  Part="1"
+AR Path="/6314CDE6/62C50742" Ref="C?"  Part="1"
+AR Path="/6314DEA9/62C50742" Ref="C52"  Part="1"
+AR Path="/6314F719/62C50742" Ref="C?"  Part="1"
+F 0 "C52" H 7040 3015 50  0000 C CNN
+F 1 "1uF" H 6980 3080 50  0000 C CNN
+F 2 "Capacitor_SMD:C_0402_1005Metric" H 7238 2925 50  0001 C CNN
+F 3 "~" H 7200 3075 50  0001 C CNN
+F 4 "C1005X5R1E105K050BE" H 7200 3075 50  0001 C CNN "PartNumber"
+F 5 "+-10%" H 7200 3075 50  0001 C CNN "Tolerance"
+F 6 "25V" H 7015 3155 50  0000 C CNN "Voltage"
+F 7 "X5R" H 7200 3075 50  0001 C CNN "Temp_Val"
+F 8 "https://www.digikey.com/en/products/detail/tdk-corporation/C1005X5R1E105K050BE/7907739" V 7200 3075 50  0001 C CNN "URL"
+	1    7200 3075
+	-1   0    0    1
+$EndComp
+$Comp
+L Device:R R?
+U 1 1 613AD852
+P 4460 4705
+AR Path="/5F71E87D/613AD852" Ref="R?"  Part="1"
+AR Path="/5F71E4A6/613AD852" Ref="R?"  Part="1"
+AR Path="/6314DEA9/613AD852" Ref="R71"  Part="1"
+F 0 "R71" V 4500 4875 50  0000 L CNN
+F 1 "160" V 4510 4450 50  0000 L CNN
+F 2 "Resistor_SMD:R_0402_1005Metric" V 4390 4705 50  0001 C CNN
+F 3 "~" H 4460 4705 50  0001 C CNN
+F 4 "1%" V 4400 4480 50  0000 L CNN "Tolerance"
+F 5 "ERJ-2RKF1600X" H 4460 4705 50  0001 C CNN "PartNumber"
+	1    4460 4705
+	0    -1   -1   0
+$EndComp
+Text Notes 4095 4580 0    20   ~ 0
+Possibly increase resistor here for less brightness
+Wire Wire Line
+	10600 2950 10600 3800
+$Comp
+L Device:C C?
+U 1 1 631AA0D8
+P 7000 2600
+AR Path="/5F71E87D/631AA0D8" Ref="C?"  Part="1"
+AR Path="/5F71E4A6/631AA0D8" Ref="C?"  Part="1"
+AR Path="/6314CDE6/631AA0D8" Ref="C?"  Part="1"
+AR Path="/6314DEA9/631AA0D8" Ref="C53"  Part="1"
+F 0 "C53" H 7160 2670 50  0000 C CNN
+F 1 "4.7uF" H 7220 2590 50  0000 C CNN
+F 2 "Capacitor_SMD:C_0402_1005Metric" H 7038 2450 50  0001 C CNN
+F 3 "~" H 7000 2600 50  0001 C CNN
+F 4 "CL05A475KP5NRNC " H 7000 2600 50  0001 C CNN "PartNumber"
+F 5 "+-10%" H 7000 2600 50  0001 C CNN "Tolerance"
+F 6 "10V" H 7200 2510 50  0000 C CNN "Voltage"
+F 7 "X5R" H 7000 2600 50  0001 C CNN "Temp_Coeff"
+F 8 "https://www.digikey.com/product-detail/en/samsung-electro-mechanics/CL05A475KP5NRNC/1276-1480-1-ND/3889566" H 7000 2600 50  0001 C CNN "URL"
+	1    7000 2600
+	1    0    0    -1
+$EndComp
+Wire Wire Line
+	7000 2750 7000 2850
+Connection ~ 7000 2850
+Wire Wire Line
+	7000 2850 6960 2850
+$Comp
+L power:GND #PWR043
+U 1 1 631B553E
+P 7000 2350
+F 0 "#PWR043" H 7000 2100 50  0001 C CNN
+F 1 "GND" H 7005 2177 50  0000 C CNN
+F 2 "" H 7000 2350 50  0001 C CNN
+F 3 "" H 7000 2350 50  0001 C CNN
+	1    7000 2350
+	-1   0    0    1
+$EndComp
+Wire Wire Line
+	7000 2350 7000 2450
 $EndSCHEMATC
