File: APT-KRIA-FMC.sch (KiCad schematic (older format))
At the start: 32 parts

Commit message: Update May --> See Update Note
Connections:
- no-connect marks 92 -> 93
Other:
- note added: "For High Speed PCB Guidelines\nRefer to page 315/347 of ug583\nTl;Dr Jog outs recommended for length matching"
- note added: "Mipi PCB guidelines on Page 203/347 of UG 583"

Commit message: Pre-Production Push
Parts:
- added TP11, TP12, TP13, TP14, TP15: TestPoint, ApotheoTech_CXP_Lib:TestPoint, symbol Connector:TestPoint
Connections:
- net FMC_3V3: now also TP13.1
- net GND: now also TP1.1
- net VCCOEN_PL_M2C: now also TP14.1
- net VCCOEN_PS_M2C: now also TP15.1
- net +5V: now reaches TP7.1
- net PS_1V8: now reaches TP4.1
- net PS_3V3: now reaches TP6.1
- net FMC_Carrier_Conn/PRSNT_M2C_B renamed FMC_Carrier_Conn/HDC18_PRSNT_M2C_B
- new net 3V8_VDD_SLVS_EC: TP11.1
- new net VADJ_FMC: TP12.1
- no-connect marks 93 -> 78
Other:
- note added: "(148.5MHz default)\n(LVDS standard)"
- note added: "Baro \n+\nAccelerometer"
- note added: "C2M is RX\n(GTR 0 and 1 for Displayport, Tx Only)"
- note added: "Camera Reset\n& GPIO"
- note added: "Clocking and I2C"
- note added: "Config"
- note added: "Displayport"
- note added: "FMC"
- note added: "For circuit board testing, must pull high\n(solder to 5V via wire for voltage monitoring)"
- note added: "HPC, \nHPB,\nHDB \nVCCO = VADJ = {1.2V to 2V}\n(Default 1.8V)"
- note added: "JTAG + Debug"
- note added: "Power"
- note added: "Power\nMonitor \n+\nFan"
- note added: "SATA"
- note added: "SD Card"
- note added: "SLVS-EC GTH\nclocking"
- note added: "SLVS-EC\nFRAMOS"
- note added: "Status and Reset"
- note added: "To ensure no conflicts with SOM I2C \nADDR (I2C1), use I2C0 for Board"
- note added: "USB 3.0"
- note added: "Unused HDA"
- note added: "Unused HDB"
- note added: "Unused HDC"
- note added: "Unused MIO"
- note added: "Unused\nHPA"
- note added: "Unused\nPS-GTR"
- note added: "VCCO = 3.3V"
- note added: "VCCO = VADJ"
- note added: "VCCO = VADJ\nMUST be 1.8V \nfor proper operation"
- note removed: "C2M is RX (GTR 0 and 1 for Displayport)"
- note removed: "IAS0"
- note removed: "To ensure no conflicts with SOM I2C \nADDR, use other MIO for I2C"
- moved on the sheet: R5, R6

Commit message: Update to Kicad 7
Parts:
- added SYM5: SYM_ESD_Small, Symbol:CE-Logo_8.5x6mm_SilkScreen, symbol Graphic:SYM_ESD_Small
- added SYM6: SYM_ESD_Small, ApotheoTech_CXP_Lib:UKCA_Logo_8_5mm, symbol Graphic:SYM_ESD_Small
Connections:
- net FMC_Carrier_Conn/HDC18_PRSNT_M2C_B renamed HDC18_PRSNT_M2C_B
Changed lines of the file:
@@
 	16500 10005 16000 10005
 $Sheet
-S 8000 4260 3500 650
+S 8000 4260 3500 840
 U 61AA736C
 F0 "Kria_Reset" 50
@@
 F13 "FMC_PG" I R 11500 4850 50
 F14 "VADJ_EN" O L 8000 4665 50
+F15 "HDC20_VADJ_ALERT" I R 11500 4920 50
+F16 "HDC19_INA226_ALERT" I R 11500 4990 50
+F17 "HDC18_PRSNT_M2C_B" I R 11500 5060 50
 $EndSheet
 Wire Wire Line
@@
 Wire Wire Line
 	7550 4665 8000 4665
+$Comp
+L Graphic:SYM_ESD_Small SYM5
+U 1 1 63BD555A
+P 5025 15705
+F 0 "SYM5" H 5165 15718 50  0000 L CNN
+F 1 "SYM_ESD_Small" H 5025 15580 50  0001 C CNN
+F 2 "Symbol:CE-Logo_8.5x6mm_SilkScreen" H 5025 15715 50  0001 C CNN
+F 3 "~" H 5025 15715 50  0001 C CNN
+	1    5025 15705
+	1    0    0    -1
+$EndComp
+$Comp
+L Graphic:SYM_ESD_Small SYM6
+U 1 1 63ADEC7E
+P 5545 15710
+F 0 "SYM6" H 5685 15723 50  0000 L CNN
+F 1 "SYM_ESD_Small" H 5545 15585 50  0001 C CNN
+F 2 "ApotheoTech_CXP_Lib:UKCA_Logo_8_5mm" H 5545 15720 50  0001 C CNN
+F 3 "~" H 5545 15720 50  0001 C CNN
+	1    5545 15710
+	1    0    0    -1
+$EndComp
+Text Label 16090 7445 0    20   ~ 0
+HDC18_PRSNT_M2C_B
+Wire Wire Line
+	11950 4920 11500 4920
+Wire Wire Line
+	11950 4990 11500 4990
+Wire Wire Line
+	11950 5060 11500 5060
+Text Label 11950 5060 2    20   ~ 0
+HDC18_PRSNT_M2C_B
+Text Label 11650 7470 0    20   ~ 0
+HDC19_INA226_ALERT
+Text Label 11650 7400 0    20   ~ 0
+HDC20_VADJ_ALERT
+Text Label 11950 4990 2    20   ~ 0
+HDC19_INA226_ALERT
+Text Label 11950 4920 2    20   ~ 0
+HDC20_VADJ_ALERT
 $EndSCHEMATC
