File: Baro_IMU.sch (KiCad schematic (older format))
At the start: 6 parts, among them U34 ICP-10111, U9 ICM-42688-P

Commit message: Update May --> See Update Note
Parts:
- removed U34: ICP-10111, ApotheoTech_CXP_Lib:ICP-10111, symbol ApotheoTech:ICP-10111
- added IC22: MS561101BA03-50, ApotheoTech_CXP_Lib:MS561101BA03-50, symbol ApotheoTech:MS561101BA03-50
Connections:
- net GND: now also IC22.3 (GND)
- net PL_3V3: now also IC22.1 (VDD)
- new net CS_MS5611: IC22.4 (CSB_1), IC22.5 (CSB_2)
- new net MODE_MS5611: IC22.2 (PS)
- new net SCL_MS5611: IC22.8 (SCLK)
- new net SDA_SDI_MS5611: IC22.7 (SDI/SDA)
- new net SDO_MS5611: IC22.6 (SDO)
Other:
- moved on the sheet: C264
Changed lines of the file:
@@
 CLK_ICM_42688
 $Comp
-L ApotheoTech:ICP-10111 U34
-U 1 1 61A6D03E
-P 7800 2200
-F 0 "U34" H 7825 2575 50  0000 C CNN
-F 1 "ICP-10111" H 7825 2484 50  0000 C CNN
-F 2 "ApotheoTech_CXP_Lib:ICP-10111" H 7800 2200 50  0001 C CNN
-F 3 "" H 7800 2200 50  0001 C CNN
-	1    7800 2200
+L power:GND #PWR0323
+U 1 1 61A70D3B
+P 7050 2100
+F 0 "#PWR0323" H 7050 1850 50  0001 C CNN
+F 1 "GND" H 7055 1927 50  0000 C CNN
+F 2 "" H 7050 2100 50  0001 C CNN
+F 3 "" H 7050 2100 50  0001 C CNN
+	1    7050 2100
 	1    0    0    -1
 $EndComp
 Wire Wire Line
-	8350 2150 8500 2150
+	8565 1560 8965 1560
+Text HLabel 8965 1560 2    50   BiDi ~ 0
+SDA_SDI_MS5611
 Wire Wire Line
-	8500 2150 8500 2350
-Wire Wire Line
-	8500 2350 8350 2350
-Wire Wire Line
-	8500 2350 8500 2500
-Connection ~ 8500 2350
-Wire Wire Line
-	7300 2050 7150 2050
-Wire Wire Line
-	7150 2050 7150 2600
+	8565 1460 8965 1460
+Text HLabel 8965 1460 2    50   Input ~ 0
+SCL_MS5611
 $Comp
-L power:GND #PWR0322
-U 1 1 61A70266
-P 8500 2600
-F 0 "#PWR0322" H 8500 2350 50  0001 C CNN
-F 1 "GND" H 8505 2427 50  0000 C CNN
-F 2 "" H 8500 2600 50  0001 C CNN
-F 3 "" H 8500 2600 50  0001 C CNN
-	1    8500 2600
-	1    0    0    -1
-$EndComp
-$Comp
-L power:GND #PWR0323
-U 1 1 61A70D3B
-P 7150 2600
-F 0 "#PWR0323" H 7150 2350 50  0001 C CNN
-F 1 "GND" H 7155 2427 50  0000 C CNN
-F 2 "" H 7150 2600 50  0001 C CNN
-F 3 "" H 7150 2600 50  0001 C CNN
-	1    7150 2600
+L ApotheoTech:MS561101BA03-50 IC22
+U 1 1 629D52A8
+P 7265 1460
+F 0 "IC22" H 7915 1725 50  0000 C CNN
+F 1 "MS561101BA03-50" H 7915 1634 50  0000 C CNN
+F 2 "ApotheoTech_CXP_Lib:MS561101BA03-50" H 8415 1560 50  0001 L CNN
+F 3 "http://www.te.com/usa-en/search.html?q=ms5611&source=header" H 8415 1460 50  0001 L CNN
+F 4 "Sensor Pressure 1.2bar Barometric SMD MS561101BA03-50, Barometric Pressure Sensor, 1200mbar 0  3.6 V Output, 8-Pin QFN" H 8415 1360 50  0001 L CNN "Description"
+F 5 "" H 8415 1260 50  0001 L CNN "Height"
+F 6 "824-MS561101BA03-50" H 8415 1160 50  0001 L CNN "Mouser Part Number"
+F 7 "https://www.mouser.co.uk/ProductDetail/Measurement-Specialties/MS561101BA03-50/?qs=%252BgKeJhng5iV%252BnCz6Qd5iDw%3D%3D" H 8415 1060 50  0001 L CNN "Mouser Price/Stock"
+F 8 "TE Connectivity" H 8415 960 50  0001 L CNN "Manufacturer_Name"
+F 9 "MS561101BA03-50" H 8415 860 50  0001 L CNN "Manufacturer_Part_Number"
+	1    7265 1460
 	1    0    0    -1
 $EndComp
@@
 L Device:C C?
 U 1 1 61A74E86
-P 8750 2250
+P 7100 1250
 AR Path="/5F71E87D/61A74E86" Ref="C?"  Part="1"
 AR Path="/5F71E4A6/61A74E86" Ref="C?"  Part="1"
@@
 AR Path="/63747F19/61A74E86" Ref="C?"  Part="1"
 AR Path="/61A5200E/61A74E86" Ref="C264"  Part="1"
-F 0 "C264" H 8590 2190 50  0000 C CNN
-F 1 "0.1uF" H 8530 2255 50  0000 C CNN
-F 2 "Capacitor_SMD:C_0402_1005Metric" H 8788 2100 50  0001 C CNN
-F 3 "~" H 8750 2250 50  0001 C CNN
-F 4 "TMK105BJ104KVHF" H 8750 2250 50  0001 C CNN "PartNumber"
-F 5 "+-10%" H 8750 2250 50  0001 C CNN "Tolerance"
-F 6 "25V" H 8565 2330 50  0000 C CNN "Voltage"
-F 7 "X5R" H 8750 2250 50  0001 C CNN "Temp_Val"
-F 8 "https://www.digikey.com/en/products/detail/TMK105BJ104KVHF/587-3808-1-ND/4811278?itemSeq=375666509" V 8750 2250 50  0001 C CNN "URL"
-	1    8750 2250
+F 0 "C264" H 6940 1190 50  0000 C CNN
+F 1 "0.1uF" H 6880 1255 50  0000 C CNN
+F 2 "Capacitor_SMD:C_0402_1005Metric" H 7138 1100 50  0001 C CNN
+F 3 "~" H 7100 1250 50  0001 C CNN
+F 4 "TMK105BJ104KVHF" H 7100 1250 50  0001 C CNN "PartNumber"
+F 5 "+-10%" H 7100 1250 50  0001 C CNN "Tolerance"
+F 6 "25V" H 6915 1330 50  0000 C CNN "Voltage"
+F 7 "X5R" H 7100 1250 50  0001 C CNN "Temp_Val"
+F 8 "https://www.digikey.com/en/products/detail/TMK105BJ104KVHF/587-3808-1-ND/4811278?itemSeq=375666509" V 7100 1250 50  0001 C CNN "URL"
+	1    7100 1250
+	1    0    0    -1
+$EndComp
+Wire Wire Line
+	7265 1460 7100 1460
+Wire Wire Line
+	7100 1460 7100 1400
+Wire Wire Line
+	7100 1100 7100 950
+$Comp
+L power:GND #PWR037
+U 1 1 629E0059
+P 7100 950
+F 0 "#PWR037" H 7100 700 50  0001 C CNN
+F 1 "GND" H 7105 777 50  0000 C CNN
+F 2 "" H 7100 950 50  0001 C CNN
+F 3 "" H 7100 950 50  0001 C CNN
+	1    7100 950
 	-1   0    0    1
 $EndComp
 Wire Wire Line
-	8750 2400 8750 2500
+	8565 1760 8700 1760
 Wire Wire Line
-	8750 2500 8500 2500
-Connection ~ 8500 2500
+	8700 1760 8700 1950
 Wire Wire Line
-	8500 2500 8500 2600
+	8700 1950 7150 1950
 Wire Wire Line
-	8350 2050 8750 2050
+	7150 1950 7150 1760
 Wire Wire Line
-	8750 2050 8750 2100
+	7150 1760 7265 1760
 Wire Wire Line
-	8750 2050 9050 2050
-Connection ~ 8750 2050
-Text GLabel 9050 2050 2    50   Input ~ 0
+	7265 1660 7050 1660
+Wire Wire Line
+	7050 1660 7050 2100
+Wire Wire Line
+	8565 1660 8965 1660
+Text HLabel 8965 1660 2    50   Output ~ 0
+SDO_MS5611
+Wire Wire Line
+	8700 1760 8965 1760
+Connection ~ 8700 1760
+Text HLabel 8965 1760 2    50   Output ~ 0
+CS_MS5611
+Wire Wire Line
+	7265 1560 6865 1560
+Text HLabel 6865 1560 0    50   BiDi ~ 0
+MODE_MS5611
+Wire Wire Line
+	7100 1460 6850 1460
+Connection ~ 7100 1460
+Text GLabel 6850 1460 0    50   Input ~ 0
 PL_3V3
-Wire Wire Line
-	7300 2250 6900 2250
-Text HLabel 6900 2250 0    50   BiDi ~ 0
-SDA_ICP_10111
-Wire Wire Line
-	7300 2350 6900 2350
-Text HLabel 6900 2350 0    50   Input ~ 0
-SCL_ICP_10111
 $EndSCHEMATC

Commit message: Pre-Production Push
Parts:
- added R44, R51: 10K, Resistor_SMD:R_0402_1005Metric, symbol Device:R
Connections:
- net PL_3V3: now also R44.1, R51.1
- net CLK_ICM_42688 renamed HDC03_CLK_ICM_42688
- net CS_ICM_42688 renamed HDC08_CS_ICM_42688
- net HDC08_CS_ICM_42688: now also R44.2
- net CS_MS5611 renamed HDC11_CS_MS5611
- net HDC11_CS_MS5611: now also R51.2
- net INT_ICM_42688 renamed HDC00_CC_INT_ICM_42688
- net MODE_MS5611 renamed HDC23_MODE_MS5611
- net SCLK_ICM_42688 renamed HDC07_SCLK_ICM_42688
- net SCL_MS5611 renamed HDC05_SCL_MS5611
- net SDA_SDI_MS5611 renamed HDC04_SDA_SDI_MS5611
- net SDI_ICM_42688 renamed HDC02_SDI_ICM_42688
- net SDO_ICM_42688 renamed HDC01_SDO_ICM_42688
- net SDO_MS5611 renamed HDC10_SDO_MS5611
Other:
- moved on the sheet: C179, C180, C263, U9

Commit message: Update to Kicad 7
Parts:
- C263: PartNumber CL21B225KAFNNNE -> GRM155R61E225KE1D
Changed lines of the file:
@@
 F 4 "+-10%" H 4700 2850 50  0001 C CNN "Tolerance"
 F 5 "25V" H 4815 2759 50  0000 L CNN "Voltage"
-F 6 "CL21B225KAFNNNE" H 4700 2850 50  0001 C CNN "PartNumber"
+F 6 "GRM155R61E225KE1D" H 4700 2850 50  0001 C CNN "PartNumber"
 	1    4700 2850
 	1    0    0    -1
