File: Kria_Reset.sch (KiCad schematic (older format))
At the start: 29 parts, among them IC17 AGLN010V5-UCG36, IC18 74AVC4T245RSVR-NT, J15 TSM-105-01-L-DV, Q19 DMN26D0UFB4-7, Q20 DMN26D0UFB4-7, Q21 DMN26D0UFB4-7, U23 SN74AXC1T45DCKR

Commit message: Update May --> See Update Note
Parts:
- removed C186, C190, C194: 0.1uF, Capacitor_SMD:C_0402_1005Metric, symbol Device:C
- removed C188, C193, C195: 0.01uF, Capacitor_SMD:C_0402_1005Metric, symbol Device:C
- removed IC17: AGLN010V5-UCG36, ApotheoTech_CXP_Lib:AGLN010V5-UCG36, symbol ApotheoTech:AGLN010V5-UCG36
- removed R156: 0, Resistor_SMD:R_0402_1005Metric, symbol Device:R
- added C44, C45: 1uF, Capacitor_SMD:C_0402_1005Metric, symbol Device:C
- added R35: 10K, Resistor_SMD:R_0402_1005Metric, symbol Device:R
- added U4: PIC18LF47K42-I-MV, ApotheoTech_CXP_Lib:PIC18LF47K42-I-MV, symbol ApotheoTech:PIC18LF47K42-I-MV
- J15: value TSM-105-01-L-DV -> 3220-10-0100-00; footprint ApotheoTech_CXP_Lib:103308-1 -> ApotheoTech_CXP_Lib:3220-10-0100-00
- S1: footprint B3U-1000P -> ApotheoTech_CXP_Lib:B3U-1000P
Connections:
- net TCK_IGLOO is gone; now on net UTIL_3V3: J15.1 (Pin_1)
- net TDI_IGLOO is gone; now on net GND: J15.9 (Pin_9)
- net TDO_IGLOO is gone; now on net GND: J15.3 (Pin_3)
- net TMS_IGLOO is gone; now on net GND: J15.5 (Pin_5)
- net CAM0_RESET_N: now also U4.35 (RD1)
- net CAM1_RESET_N: now also U4.40 (RC6)
- net CC_PL_PGOOD_LS_3V3: now also U4.20 (RA3)
- net CC_PS_PGOOD_LS_3V3: now also U4.19 (RA2)
- net GND: now also C44.1, C45.1, U4.27 (VSS), U4.41 (EPAD), U4.6 (VSS); no longer J15.10 (Pin_10), J15.2 (Pin_2)
- net HDB03_CAM0_RESET_N: now also U4.4 (RD6)
- net HDB04_CAM1_RESET_N: now also U4.5 (RD7)
- net MIO43_SD_RESET_3V3: now also U4.29 (RA6)
- net MIO44_USB_RESET_3V3: now also U4.28 (RA7)
- net PS_POR_B_3V3: now also U4.31 (RC1)
- net PS_POR_B_3V3_L: now also U4.34 (RD0)
- net PS_POR_B_DIR: now also U4.32 (RC2)
- net RST_BUTTON_N: now also U4.37 (RD3)
- net SD_RESET_N: now also U4.36 (RD2)
- net USB_RESET_OUT_3V3: now also U4.30 (RC0)
- net UTIL_3V3: now also C44.2, C45.2, R35.2, U4.26 (VDD), U4.7 (VDD); no longer J15.6 (Pin_6)
- net ICSPCLK: now reaches J15.4 (Pin_4)
- net ICSPCLK: now also U4.14 (ICSPCLK/RB6)
- net PG_FMC_SHORT renamed VADJ_FMC_PG_MCU
- net VADJ_FMC_PG_MCU: now also U4.3 (RD5)
- net TRST_IGLOO: no longer names the net of J15.8 (Pin_8)
- net VPUMP_IGLOO: no longer names the net of J15.7 (Pin_7)
- new net FMC_SCL: U4.33 (RC3/SCL1)
- new net FMC_SDA: U4.38 (RC4/SDA1)
- new net ICSPDAT: J15.6 (Pin_6), U4.15 (ICSPDAT/RB7)
- new net MCLR: J15.10 (Pin_10), R35.1, U4.16 (MCLR)
- new net VADJ_SCL: U4.9 (RB1/SCL2)
- new net VADJ_SDA: U4.10 (RB2/SDA2)
- no-connect marks 8 -> 18
Other:
- note added: "* SD reset is 3.3V nominal, no change\n* Raspberry Pi Resets are 3.3V nominal, no change\n* USB reset is 1.8V nominal,"
- note added: "CORTEX JTAG/SWD (10 pin mini)"
- note added: "Does PGC mean ICSPCLK?\nDoes PGD mean ICSPDAT?\n\nRefering to sheet 8/9 for Curiosity HPC for a reference pinout (RB7 for data, RB6 for clock)"
- note added: "Note CC_P*_PGOOD is 5V high (when high CC_P*_PGOOD_LS is low\n(inverse relationship with CC_PL_GOOD)"
- note added: "PIC18LF47K42-I/MV Reset Pinout"
- note added: "PIC18LF47K42-I/MV Reset for Kria Carrier"
- note added: "PS_POR_B"
- note added: "Refer to ICD4/PICkit 4 Target Adapter Board\nCortex JTAG/SWD (10 pin mini) which this is based off of\n"
- note added: "Refer to page 11/842 of PIC datasheet\nfor SCL2 (pins 9, 10 for 40 pin UQFN)"
- note added: "Refer to page 12/842 of PIC datasheet \nfor SCL1 (pins 33 for SCL, pins 38 for SDA)"
- note removed: "* SD reset is 3.3V nominal, no change\n* Raspberry Pi Resets are 3.3V nominal, no change\n* USB reset is 1.8V nominal, must provide voltage level converion via MOSFET and resistor pullup or using TI voltage level converter"
- note removed: "Crystal for IGLOO"
- note removed: "Filter for VCCO and VJTAG"
- note removed: "IGLOO 1V5 for Core Operation"
- note removed: "IGLOO Nano JTAG Connector (FlashPro4)"
- note removed: "IGLOO Nano Reset Pinout"
- note removed: "IGLOO Nano Reset for Kria Carrier"
- note removed: "IGLOO needs a 3.3V LVCMOS crystal\nChose 54MHz that is from the clock generator we have on board already\n"
- note removed: "Note CC_P*_PGOOD is 5V high (when high CC_P*_PGOOD_LS is low\n(inverse relationship in IGLOO code) \nThus, for FPGA code must be when !CC_P*_GOOD for logic"
- note removed: "Power VCORE"
- note removed: "Question: Does IGLOO Nano program via USB or JTAG?\nFigure out ABCD correct pinout, if JTAG needed,\ncan use bus B for IGLOO JTAG with similar pinout\nto Xilinx\nA: IGLOO is via JTAG like Xilinx, must use 10 pin connector\nin conjunction with the B bus for flexibility in using the\nprogrammer, and the FT4232HL\nTRST is active low, pulldown outside of FPGA is needed"
- note removed: "Will use FLASHPRO4 (3.3V compatible)\n* IGLOO Nano for reset\n* use JTAG to program IGLOO Nano\n*3.3V compatible pins\n* Note we don't use Program Mode (pin 4)\nAnd this must not be connected"
- moved on the sheet: C181, C182, C183, C184, C185, C187, C189, C191, C192, IC18, J15, Q19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

Commit message: Pre-Production Push
Parts:
- added R42, R43: 10K, Resistor_SMD:R_0402_1005Metric, symbol Device:R
- added R52: 4.7K, Resistor_SMD:R_0402_1005Metric, symbol Device:R
- R159: value 4.7K -> DNP; DNP (none) -> DNP; DNP_Val (none) -> 4.7K
- R35: value 10K -> 100K; PartNumber ERJ-2RKF1002X -> CRCW0402100KFKEDHP; Power 1/10W -> 1/5W; URL https://www.digikey.com/en/products/detail/panasonic-electr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 -> (none)
Connections:
- net GND: now also R52.1
- net PS_POR_B_3V3_L: now also R52.2
- net UTIL_3V3: now also R42.1, R43.1
- net VADJ_EN: now reaches U4.11 (RB3)
- net HDB03_CAM0_RESET_N renamed HDC14_CAM0_RESET_N
- net HDC14_CAM0_RESET_N: now also R42.2
- net HDB04_CAM1_RESET_N renamed HDC06_CAM1_RESET_N
- net HDC06_CAM1_RESET_N: now also R43.2
- net MIO43_SD_RESET_3V3 renamed MIO43_SD_RESET_3V3_N
- net MIO44_USB_RESET_3V3 renamed MIO44_USB_RESET_3V3_N
- net USB_RESET_OUT_3V3 renamed USB_RESET_OUT_3V3_N
- no-connect marks 18 -> 17
Other:
- note added: "PS_POR is pulled up 4.7K to 1.8V on SOM"
- note added: "Place all *_N pins as high (1) when not in reset"
Changed lines of the file:
@@
 $Descr A3 16535 11693
 encoding utf-8
-Sheet 9 20
+Sheet 8 20
 Title "IGLOO nano Reset for Kria Carrier"
 Date "2022-01-04"
@@
 	9700 6500 10875 6500
 Text Label 10875 6500 2    50   ~ 0
-MIO43_SD_RESET_3V3
+MIO43_SD_RESET_3V3_N
 Text Label 6045 2850 2    50   ~ 0
-MIO43_SD_RESET_3V3
+MIO43_SD_RESET_3V3_N
 Wire Wire Line
 	9700 6175 10875 6175
 Text Label 10875 6175 2    50   ~ 0
-MIO44_USB_RESET_3V3
+MIO44_USB_RESET_3V3_N
 Text Label 6045 2955 2    50   ~ 0
-MIO44_USB_RESET_3V3
+MIO44_USB_RESET_3V3_N
 Text Label 6045 2750 2    50   ~ 0
-USB_RESET_OUT_3V3
+USB_RESET_OUT_3V3_N
 Text Label 10875 6825 2    50   ~ 0
-USB_RESET_OUT_3V3
+USB_RESET_OUT_3V3_N
 Wire Wire Line
 	9700 6825 10875 6825
@@
 	5095 3150 6045 3150
 NoConn ~ 8300 7150
-Text HLabel 2330 3045 0    50   Input ~ 0
-HDB03_CAM0_RESET_N
+Text HLabel 1450 3045 0    50   Input ~ 0
+HDC14_CAM0_RESET_N
 Text Label 4645 1910 3    25   ~ 0
 PS_POR_B_3V3
 Text Label 4545 1910 3    25   ~ 0
 PS_POR_B_DIR
-Text HLabel 10550 9500 2    50   BiDi ~ 0
-PS_POR_B
-Text GLabel 9920 9050 0    50   Input ~ 0
-PS_1V8
-Wire Wire Line
-	10000 9050 9920 9050
-Wire Wire Line
-	10000 9050 10000 9150
-$Comp
-L Device:R R?
-U 1 1 61DC3C3D
-P 10000 9300
-AR Path="/5F71E87D/61DC3C3D" Ref="R?"  Part="1"
-AR Path="/62C99A69/61DC3C3D" Ref="R?"  Part="1"
-AR Path="/61AA736C/61DC3C3D" Ref="R159"  Part="1"
-F 0 "R159" H 10070 9391 50  0000 L CNN
-F 1 "4.7K" H 10070 9300 50  0000 L CNN
-F 2 "Resistor_SMD:R_0402_1005Metric" V 9930 9300 50  0001 C CNN
-F 3 "~" H 10000 9300 50  0001 C CNN
-F 4 "1%" H 10070 9209 50  0000 L CNN "Tolerance"
-F 5 "CRCW04024K70FKED" H 10000 9300 50  0001 C CNN "PartNumber"
-	1    10000 9300
-	1    0    0    -1
-$EndComp
-$Comp
-L power:GND #PWR?
-U 1 1 61DC3C35
-P 10000 10250
-AR Path="/6314F1AA/61DC3C35" Ref="#PWR?"  Part="1"
-AR Path="/61AA736C/61DC3C35" Ref="#PWR0217"  Part="1"
-F 0 "#PWR0217" H 10000 10000 50  0001 C CNN
-F 1 "GND" H 10005 10077 50  0000 C CNN
-F 2 "" H 10000 10250 50  0001 C CNN
-F 3 "" H 10000 10250 50  0001 C CNN
-	1    10000 10250
-	1    0    0    -1
-$EndComp
-Wire Wire Line
-	10000 10150 10000 10250
-$Comp
-L ApotheoTech:DMN26D0UFB4-7 Q?
-U 1 1 61DC3C2E
-P 9500 9850
-AR Path="/6314F1AA/61DC3C2E" Ref="Q?"  Part="1"
-AR Path="/61AA736C/61DC3C2E" Ref="Q21"  Part="1"
-F 0 "Q21" H 10130 9903 60  0000 L CNN
-F 1 "DMN26D0UFB4-7" H 10130 9797 60  0000 L CNN
-F 2 "ApotheoTech_CXP_Lib:DMN26D0UFB4-7" H 10000 9350 60  0001 C CNN
-F 3 "" H 9500 9850 60  0000 C CNN
-	1    9500 9850
-	1    0    0    -1
-$EndComp
 $Comp
 L power:GND #PWR0213
@@
 	6130 9350 6070 9350
 Connection ~ 6070 9350
-Wire Wire Line
-	6070 9170 6070 9350
-Text Notes 11430 9290 0    79   ~ 0
+Text Notes 7740 8900 0    79   ~ 0
 Pull up, DIR high is translation from A to B\nWant POR_B to be controlled by carrier card,\nit is held in reset until PS side is good\nRefer to p age 24 of UG1089\nOnce CC_PS is good, check the PS_POR_B\nto reset all PS reliant domains
 Wire Wire Line
@@
 	6100 9850 5970 9850
 Wire Wire Line
-	6100 9750 5670 9750
-Wire Wire Line
 	6500 9350 6430 9350
 $Comp
@@
 	1    0    0    -1
 $EndComp
-Text Label 8800 9850 0    50   ~ 0
-PS_POR_B_3V3_L
-Wire Wire Line
-	8800 9850 9500 9850
-Wire Wire Line
-	10000 9450 10000 9500
-Wire Wire Line
-	10550 9500 10000 9500
-Connection ~ 10000 9500
-Wire Wire Line
-	10000 9500 10000 9550
 Text Label 4350 1910 3    25   ~ 0
 PS_POR_B_3V3_L
@@
 Wire Wire Line
 	4250 2300 4250 2110
-Wire Wire Line
-	3300 3045 2330 3045
 Wire Wire Line
 	2355 3345 3300 3345
@@
 AR Path="/61AA736C/628F3D2A" Ref="R35"  Part="1"
 F 0 "R35" H 11370 2791 50  0000 L CNN
-F 1 "10K" H 11370 2700 50  0000 L CNN
+F 1 "100K" H 11370 2700 50  0000 L CNN
 F 2 "Resistor_SMD:R_0402_1005Metric" V 11230 2700 50  0001 C CNN
 F 3 "~" H 11300 2700 50  0001 C CNN
 F 4 "1%" H 11370 2609 50  0000 L CNN "Tolerance"
-F 5 "1/10W" H 11300 2700 50  0001 C CNN "Power"
-F 6 "ERJ-2RKF1002X" H 11300 2700 50  0001 C CNN "PartNumber"
-F 7 "https://www.digikey.com/en/products/detail/panasonic-electronic-components/ERJ-2RKF1002X/192073" H 11300 2700 50  0001 C CNN "URL"
+F 5 "1/5W" H 11300 2700 50  0001 C CNN "Power"
+F 6 "CRCW0402100KFKEDHP" H 11300 2700 50  0001 C CNN "PartNumber"
 	1    11300 2700
 	1    0    0    -1
@@
 	3850 2300 3850 2000
 NoConn ~ 3850 2000
-Wire Wire Line
-	3300 3145 2330 3145
-Text HLabel 2330 3145 0    50   Input ~ 0
-HDB04_CAM1_RESET_N
+Text HLabel 1450 3145 0    50   Input ~ 0
+HDC06_CAM1_RESET_N
 Wire Wire Line
 	3300 2950 3000 2950
@@
 Wire Wire Line
 	3755 4100 3755 4400
-NoConn ~ 3755 4400
 Wire Wire Line
 	3855 4100 3855 4400
@@
 	3955 4100 3955 4400
 NoConn ~ 3955 4400
+$Comp
+L Device:R R?
+U 1 1 63D47F9C
+P 1500 2700
+AR Path="/5F71E87D/63D47F9C" Ref="R?"  Part="1"
+AR Path="/6314F1AA/63D47F9C" Ref="R?"  Part="1"
+AR Path="/6314F719/63D47F9C" Ref="R?"  Part="1"
+AR Path="/61AA736C/63D47F9C" Ref="R42"  Part="1"
+F 0 "R42" H 1570 2791 50  0000 L CNN
+F 1 "10K" H 1570 2700 50  0000 L CNN
+F 2 "Resistor_SMD:R_0402_1005Metric" V 1430 2700 50  0001 C CNN
+F 3 "~" H 1500 2700 50  0001 C CNN
+F 4 "1%" H 1570 2609 50  0000 L CNN "Tolerance"
+F 5 "1/10W" H 1500 2700 50  0001 C CNN "Power"
+F 6 "ERJ-2RKF1002X" H 1500 2700 50  0001 C CNN "PartNumber"
+F 7 "https://www.digikey.com/en/products/detail/panasonic-electronic-components/ERJ-2RKF1002X/192073" H 1500 2700 50  0001 C CNN "URL"
+	1    1500 2700
+	1    0    0    -1
+$EndComp
+$Comp
+L Device:R R?
+U 1 1 63D4FE45
+P 1800 2700
+AR Path="/5F71E87D/63D4FE45" Ref="R?"  Part="1"
+AR Path="/6314F1AA/63D4FE45" Ref="R?"  Part="1"
+AR Path="/6314F719/63D4FE45" Ref="R?"  Part="1"
+AR Path="/61AA736C/63D4FE45" Ref="R43"  Part="1"
+F 0 "R43" H 1870 2791 50  0000 L CNN
+F 1 "10K" H 1870 2700 50  0000 L CNN
+F 2 "Resistor_SMD:R_0402_1005Metric" V 1730 2700 50  0001 C CNN
+F 3 "~" H 1800 2700 50  0001 C CNN
+F 4 "1%" H 1870 2609 50  0000 L CNN "Tolerance"
+F 5 "1/10W" H 1800 2700 50  0001 C CNN "Power"
+F 6 "ERJ-2RKF1002X" H 1800 2700 50  0001 C CNN "PartNumber"
+F 7 "https://www.digikey.com/en/products/detail/panasonic-electronic-components/ERJ-2RKF1002X/192073" H 1800 2700 50  0001 C CNN "URL"
+	1    1800 2700
+	1    0    0    -1
+$EndComp
+Text GLabel 1300 2400 0    50   Input ~ 0
+UTIL_3V3
+Wire Wire Line
+	1300 2400 1500 2400
+Wire Wire Line
+	1500 2400 1500 2550
+Wire Wire Line
+	1500 2400 1800 2400
+Wire Wire Line
+	1800 2400 1800 2550
+Connection ~ 1500 2400
+Wire Wire Line
+	1450 3045 1500 3045
+Wire Wire Line
+	1500 2850 1500 3045
+Connection ~ 1500 3045
+Wire Wire Line
+	1500 3045 3300 3045
+Wire Wire Line
+	1800 2850 1800 3145
+Wire Wire Line
+	1800 3145 3300 3145
+Wire Wire Line
+	1800 3145 1450 3145
+Connection ~ 1800 3145
+Text Notes 5360 2630 0    50   ~ 0
+Place all *_N pins as high (1) when not in reset
+Text HLabel 3755 4400 3    50   Output ~ 0
+VADJ_EN
+Wire Wire Line
+	10000 9500 10000 9550
+Wire Wire Line
+	10550 9500 10000 9500
+Connection ~ 10000 9500
+Wire Wire Line
+	10000 9450 10000 9500
+Wire Wire Line
+	8800 9850 9250 9850
+Text Label 8800 9850 0    50   ~ 0
+PS_POR_B_3V3_L
+$Comp
+L ApotheoTech:DMN26D0UFB4-7 Q?
+U 1 1 61DC3C2E
+P 9500 9850
+AR Path="/6314F1AA/61DC3C2E" Ref="Q?"  Part="1"
+AR Path="/61AA736C/61DC3C2E" Ref="Q21"  Part="1"
+F 0 "Q21" H 10130 9903 60  0000 L CNN
+F 1 "DMN26D0UFB4-7" H 10130 9797 60  0000 L CNN
+F 2 "ApotheoTech_CXP_Lib:DMN26D0UFB4-7" H 10000 9350 60  0001 C CNN
+F 3 "" H 9500 9850 60  0000 C CNN
+	1    9500 9850
+	1    0    0    -1
+$EndComp
+Wire Wire Line
+	10000 10150 10000 10250
+$Comp
+L power:GND #PWR?
+U 1 1 61DC3C35
+P 10000 10250
+AR Path="/6314F1AA/61DC3C35" Ref="#PWR?"  Part="1"
+AR Path="/61AA736C/61DC3C35" Ref="#PWR0217"  Part="1"
+F 0 "#PWR0217" H 10000 10000 50  0001 C CNN
+F 1 "GND" H 10005 10077 50  0000 C CNN
+F 2 "" H 10000 10250 50  0001 C CNN
+F 3 "" H 10000 10250 50  0001 C CNN
+	1    10000 10250
+	1    0    0    -1
+$EndComp
+Wire Wire Line
+	10000 9050 10000 9150
+Wire Wire Line
+	10000 9050 9920 9050
+Text GLabel 9920 9050 0    50   Input ~ 0
+PS_1V8
+Text HLabel 10550 9500 2    50   BiDi ~ 0
+PS_POR_B
+Wire Wire Line
+	6100 9750 5670 9750
+Wire Wire Line
+	6070 9170 6070 9350
+$Comp
+L Device:R R?
+U 1 1 61DC3C3D
+P 10000 9300
+AR Path="/5F71E87D/61DC3C3D" Ref="R?"  Part="1"
+AR Path="/62C99A69/61DC3C3D" Ref="R?"  Part="1"
+AR Path="/61AA736C/61DC3C3D" Ref="R159"  Part="1"
+F 0 "R159" H 10070 9391 50  0000 L CNN
+F 1 "DNP" H 10070 9300 50  0000 L CNN
+F 2 "Resistor_SMD:R_0402_1005Metric" V 9930 9300 50  0001 C CNN
+F 3 "~" H 10000 9300 50  0001 C CNN
+F 4 "1%" H 10070 9209 50  0000 L CNN "Tolerance"
+F 5 "CRCW04024K70FKED" H 10000 9300 50  0001 C CNN "PartNumber"
+F 6 "DNP" H 10000 9300 50  0000 C CNN "DNP"
+F 7 "4.7K" H 10000 9300 50  0001 C CNN "DNP_Val"
+	1    10000 9300
+	1    0    0    -1
+$EndComp
+$Comp
+L power:GND #PWR044
+U 1 1 6348FEC5
+P 9250 10350
+F 0 "#PWR044" H 9250 10100 50  0001 C CNN
+F 1 "GND" H 9255 10177 50  0000 C CNN
+F 2 "" H 9250 10350 50  0001 C CNN
+F 3 "" H 9250 10350 50  0001 C CNN
+	1    9250 10350
+	1    0    0    -1
+$EndComp
+Wire Wire Line
+	9250 10350 9250 10230
+Wire Wire Line
+	9250 9930 9250 9850
+$Comp
+L Device:R R?
+U 1 1 6348FECF
+P 9250 10080
+AR Path="/5F71E87D/6348FECF" Ref="R?"  Part="1"
+AR Path="/5F71E4A6/6348FECF" Ref="R?"  Part="1"
+AR Path="/61AA736C/6348FECF" Ref="R52"  Part="1"
+F 0 "R52" H 9320 10171 50  0000 L CNN
+F 1 "4.7K" H 9320 10080 50  0000 L CNN
+F 2 "Resistor_SMD:R_0402_1005Metric" V 9180 10080 50  0001 C CNN
+F 3 "~" H 9250 10080 50  0001 C CNN
+F 4 "1%" H 9320 9989 50  0000 L CNN "Tolerance"
+F 5 "CRCW04024K70FKED" H 9250 10080 50  0001 C CNN "PartNumber"
+	1    9250 10080
+	-1   0    0    1
+$EndComp
+Connection ~ 9250 9850
+Wire Wire Line
+	9250 9850 9500 9850
+Text Notes 10505 9235 0    50   ~ 0
+PS_POR is pulled up 4.7K to 1.8V on SOM
 $EndSCHEMATC
