File: Micro_SD.sch (KiCad schematic (older format))
At the start: 22 parts, among them IC6 PI4ULS3V4857GEAEX, J6 502570-0893, Q8 DMN26D0UFB4-7, Q9 FDN336P

Commit message: Update May --> See Update Note
Other:
- note added: "Refer to page 195/347 UG583\n30 Ohm Reistor should be placed near the Zynq MPSOC MIO pins\n"
Changed lines of the file:
@@
 $Descr A4 11693 8268
 encoding utf-8
-Sheet 6 20
+Sheet 4 20
 Title "SD 3.0 Card"
 Date "2022-01-04"
@@
 Wire Wire Line
 	9030 2515 9030 2815
+Text Notes 1755 5335 0    50   ~ 0
+Refer to page 195/347 UG583\n30 Ohm Reistor should be placed near the Zynq MPSOC MIO pins\n
 $EndSCHEMATC

Commit message: Pre-Production Push
Other:
- note added: "Note, pinout correct here for Q9,\nBut drawing of FET is incorrect, \n2 is Source, and 3 is drain"
Changed lines of the file:
@@
 Text Notes 1755 5335 0    50   ~ 0
 Refer to page 195/347 UG583\n30 Ohm Reistor should be placed near the Zynq MPSOC MIO pins\n
+Text Notes 9350 2275 0    50   ~ 0
+Note, pinout correct here for Q9,\nBut drawing of FET is incorrect, \n2 is Source, and 3 is drain
 $EndSCHEMATC

Commit message: Update to Kicad 7
Parts:
- C81: PartNumber CL21B225KAFNNNE -> GRM155R61E225KE1D
Changed lines of the file:
@@
 F 4 "+-10%" H 5980 3655 50  0001 C CNN "Tolerance"
 F 5 "25V" H 6095 3564 50  0000 L CNN "Voltage"
-F 6 "CL21B225KAFNNNE" H 5980 3655 50  0001 C CNN "PartNumber"
+F 6 "GRM155R61E225KE1D" H 5980 3655 50  0001 C CNN "PartNumber"
 	1    5980 3655
 	1    0    0    -1
